Commit message: Add plugins for camera and Diff

File: Classic/src/hellobot/hellobot_specs/urdf/hellobot.xacro (robot description, xacro)
@@ -1,19 +1,8 @@
 <?xml version='1.0'?>
 <robot name="hellobot" xmlns:xacro="http://www.ros.org/wiki/xacro">
-    <material name="blue">
-        <color rgba="0.1 0.1 0.9 1"/>
-      </material>
-      <material name="white">
-        <color rgba="1 1 1 1"/>
-      </material>
-      <material name="green">
-        <color rgba="0 1 0 1"/>
-      </material>
-      <material name="black">
-        <color rgba="0 0 0 1"/>
-      </material>
-      <material name="yellow">
-        <color rgba="1 0 1 1"/>
-      </material>
+    <xacro:include filename="$(find hellobot_specs)/urdf/materials.xacro"/>
+    <xacro:include filename="$(find hellobot_specs)/urdf/hellobot.gazebo.xacro"/>
+    <xacro:property name="cameraSize" value="0.05"/>
+    <xacro:property name="cameraMass" value="0.1"/>
       <link name="base_footprint" />
     <joint name="base_footprint_joint" type="fixed">
@@ -41,4 +30,5 @@
       <geometry>
         <box size=".4 .2 .1"/>
+        <!-- <mesh filename="file://$(find hellobot_specs)/meshes/fixed_torta.dae" /> -->
       </geometry>
       <material name="black"/>
@@ -65,4 +55,5 @@
         <sphere radius="0.05"/>
       </geometry>
+      <material name="green">   </material>
     </visual>
     <collision name='caster_front_collision'>
@@ -87,4 +78,5 @@
         <sphere radius="0.05"/>
       </geometry>
+      <material name="green">   </material>
     </visual>
   </link>
@@ -155,3 +147,31 @@
     <joint_properties damping="0.0" friction="0.0"/>
   </joint>
+  <!-- Camera -->
+  <link name="camera_link">
+    <collision>
+      <origin xyz="0 0 0" rpy="0 0 0"/>
+      <geometry>
+        <box size="${cameraSize} ${cameraSize} ${cameraSize}"/>
+      </geometry>
+    </collision>
+    <visual>
+      <origin xyz="0 0 0" rpy="0 0 0"/>
+      <geometry>
+        <box size="${cameraSize} ${cameraSize} ${cameraSize}"/>
+      </geometry>
+      <material name="green"/>
+    </visual>
+    <inertial>
+      <mass value="${cameraMass}" />
+      <origin xyz="0 0 0" rpy="0 0 0"/>
+      <box_inertia m="${cameraMass}" x="${cameraSize}" y="${cameraSize}" z="${cameraSize}" />
+      <inertia ixx="1e-6" ixy="0" ixz="0" iyy="1e-6" iyz="0" izz="1e-6" />
+    </inertial>
+  </link>
+  <joint name="camera_joint" type="fixed">
+    <axis xyz="0 1 0" />
+    <origin xyz=".2 0 0" rpy="0 0 0"/>
+    <parent link="chassis"/>
+    <child link="camera_link"/>
+  </joint>
 </robot>
